Commit message: Fix some errors describing Robot2R

File: models/double-pendulum.urdf (robot description, URDF)
Before this commit: robot robot2R-planar, 3 links, 2 joints
Joints:
- joint join1: origin xyz=0 0 0 rpy=0 0 0 -> xyz=0.0 0 0 rpy=0 0 0
- joint join2: origin xyz=0 0 0 rpy=0 0 0 -> xyz=0.5 0 0 rpy=0 0 0
